File: camprj_kicad/IMU.sch (KiCad schematic (older format))
At the start: 10 parts, among them U7 ADP150AUJZ-3.3-R7, U8 FIS1100, U9 ADP150AUJZ-1.8-R7

Commit message: Final Delivery
Parts:
- U7: MPN (none) -> ADP150AUJZ-3.3-R7
- U8: MPN (none) -> FIS1100
- U9: MPN (none) -> ADP150AUJZ-1.8-R7
Changed lines of the file:
@@
 Date "2017-07-06"
 Rev "1"
-Comp "D-HEST ETH Zurich"
+Comp "MHSL ETH Zurich"
 Comment1 "Geethan Karunaratne"
 Comment2 ""
@@
 F 3 "http://www.mouser.com/ds/2/308/FIS1100-1119815.pdf" H 4600 2400 50  0001 C CNN
 F 4 "http://eu.mouser.com/ProductDetail/Fairchild-Semiconductor/FIS1100/?qs=Pve5fMu%2FDEuZUDX%2Fo6J%252b1g%3D%3D" H 4500 3200 60  0001 C CNN "Buy Link"
+F 5 "FIS1100" H 4500 3200 60  0001 C CNN "MPN"
 	1    4500 3200
 	1    0    0    -1
@@
 F 3 "http://www.mouser.com/ds/2/609/ADP150-773560.pdf" H 4500 1150 60  0001 C CNN
 F 4 "http://eu.mouser.com/ProductDetail/Analog-Devices/ADP150AUJZ-33-R7/?qs=WIvQP4zGanjNlX1MqHWsFA%3D%3D" H 4500 1150 60  0001 C CNN "Buy Link"
+F 5 "ADP150AUJZ-3.3-R7" H 4500 1150 60  0001 C CNN "MPN"
 	1    4500 1150
 	1    0    0    -1
@@
 F 3 "http://www.mouser.com/ds/2/609/ADP150-773560.pdf" H 7050 1150 60  0001 C CNN
 F 4 "http://eu.mouser.com/ProductDetail/Analog-Devices/ADP150AUJZ-18-R7/?qs=WIvQP4zGanj6me7Xqf%252bL8w%3D%3D" H 7050 1150 60  0001 C CNN "Buy Link"
+F 5 "ADP150AUJZ-1.8-R7" H 7050 1150 60  0001 C CNN "MPN"
 	1    7050 1150
 	1    0    0    -1
