File: camprj_kicad/power_supply.sch (KiCad schematic (older format))
At the start: 15 parts, among them J2 USB_OTG, U16 BQ24075RGTR

Commit message: Board design: component placement done
Parts:
- added Q1: DMMT5401, TO_SOT_Packages_SMD:SOT-23-6_Handsoldering, symbol DMMT5401
- added Q2: DMG2305UX, TO_SOT_Packages_SMD:SOT-23, symbol Q_PMOS_GSD
- added RR1: 10K, Resistors_SMD:R_0603_HandSoldering, symbol R
- added RR2: 47K, Resistors_SMD:R_0603_HandSoldering, symbol R
- JP1: value SPARKFUN-CONNECTORS_JST_2MM_MALE -> JST_2MM_MALE; symbol SPARKFUN-CONNECTORS_JST_2MM_MALE -> SPARKFUN-CONNECTORS_JST_2MM_MALE-RESCUE-camprj_kicad
Connections:
- net GND: now also RR1.2, RR2.2
- net +5V: no longer names the net of C41.1, R16.1, R17.1, U16.10 (OUT), U16.11 (OUT), U16.5 (EN2)
- net +5V: now also Q1.5 (E2), Q2.3 (D)
- new net: Q1.2 (B1), Q1.3 (B2), Q1.4 (C2), RR1.1
- new net: Q1.1 (C1), Q2.1 (G), RR2.1
- new net V5_0: Q1.6 (E1), Q2.2 (S)
Other:
- note added: "Ideal Diode\nBackpowering saftey circuit\n"

Commit message: Final Delivery
Parts:
- J2: MPN (none) -> 629105150521
- JP1: MPN (none) -> BM02B-CPTK-1A-TB
- Q1: MPN (none) -> DMMT5401-7-F
- Q2: MPN (none) -> DMG2305UX-13
- S1: MPN (none) -> 1825282-1
- U16: MPN (none) -> BQ24075RGTR
Changed lines of the file:
@@
 Date "2017-07-07"
 Rev "1"
-Comp "D-HEST ETH Zurich"
+Comp "MHSL ETH Zurich"
 Comment1 "Geethan Karunaratne"
 Comment2 ""
@@
 F 3 "http://www.ti.com/lit/ds/symlink/bq24075.pdf" H 5000 3850 60  0001 C CNN
 F 4 "http://eu.mouser.com/ProductDetail/Texas-Instruments/BQ24075RGTR/?qs=sGAEpiMZZMs7zYnFw9eWkqY9KdX9yrFF" H 5000 3850 60  0001 C CNN "Buying Link"
+F 5 "BQ24075RGTR" H 5000 3850 60  0001 C CNN "MPN"
 	1    5000 3850
 	1    0    0    -1
@@
 F 3 "http://www.mouser.com/ds/2/445/629105150521-469306.pdf" H 1400 1050 50  0001 C CNN
 F 4 "http://www.mouser.ch/ProductDetail/Wurth-Electronics/629105150521/?qs=a9WhcLg8qCzXiH7kZP8GRQ%3d%3d" H 1250 1100 60  0001 C CNN "Buy Link"
+F 5 "629105150521" H 1250 1100 60  0001 C CNN "MPN"
 	1    1250 1100
 	1    0    0    -1
@@
 F 4 "http://www.mouser.ch/ProductDetail/JST-Automotive/BM02B-CPTK-1A-TB/?qs=sGAEpiMZZMs7eK6h2EBtKpZPrn2bvQ1TQstUUrXc%2ftY%3d" H 3150 1000 60  0001 C CNN "Buy Link"
 F 5 "https://www.sparkfun.com/products/13813" H 3150 1000 60  0001 C CNN "Battery"
+F 6 "BM02B-CPTK-1A-TB" H 3150 1000 60  0001 C CNN "MPN"
 	1    3150 1000
 	0    -1   -1   0
@@
 F 3 "http://www.te.com/commerce/DocumentDelivery/DDEController?Action=srchrtrv&DocNm=1825282&DocType=Customer+Drawing&DocLang=English" H 5150 1250 60  0001 C CNN
 F 4 "https://www.digikey.com/product-detail/en/te-connectivity-alcoswitch-switches/1825282-1/450-1635-ND/1308844" H 5150 1250 60  0001 C CNN "Buy Link"
+F 5 "1825282-1" H 5150 1250 60  0001 C CNN "MPN"
 	1    5150 1250
 	1    0    0    -1
@@
 F 3 "https://www.diodes.com/assets/Datasheets/DMG2305UX.pdf" H 8900 3450 50  0001 C CNN
 F 4 "http://www.mouser.ch/ProductDetail/Diodes-Incorporated/DMG2305UX-13/?qs=L1DZKBg7t5Hgw5KN3G2IRg==" H 8900 3450 60  0001 C CNN "Buy Link"
+F 5 "DMG2305UX-13" H 8900 3450 60  0001 C CNN "MPN"
 	1    8900 3450
 	0    -1   -1   0
@@
 F 3 "https://www.diodes.com/assets/Datasheets/ds30437.pdf" H 8800 3950 50  0001 C CNN
 F 4 "http://www.mouser.ch/ProductDetail/Diodes-Incorporated/DMMT5401-7-F/?qs=hiZRsJxw0h3f7LzTPwvEFQ==" H 8900 4050 60  0001 C CNN "Buy Link"
+F 5 "DMMT5401-7-F" H 8600 3900 60  0001 C CNN "MPN"
 	2    8600 3900
 	-1   0    0    1
@@
 F 3 "https://www.diodes.com/assets/Datasheets/ds30437.pdf" H 9400 3950 50  0001 C CNN
 F 4 "http://www.mouser.ch/ProductDetail/Diodes-Incorporated/DMMT5401-7-F/?qs=hiZRsJxw0h3f7LzTPwvEFQ==" H 9500 4050 60  0001 C CNN "Buy Link"
+F 5 "DMMT5401-7-F" H 9200 3900 60  0001 C CNN "MPN"
 	1    9200 3900
 	1    0    0    1
