File: camprj_kicad/single_led_drive.sch (KiCad schematic (older format))
At the start: 11 parts, among them U11 MAX1561

Commit message: Board design: component placement done
Parts:
- removed D7: B340A, Myfootprints:D_SMA_Handsoldering_AC, symbol LEPTONCUSTOM_DIODE-SCHOTTKY-B340A
- added D12: CMDSH2-3, Diodes_SMD:D_SOD-323_HandSoldering, symbol CMDSH2-3
Connections:
- net at C26.1, D8.2 (A), U11.1 (OUT): now also D12.2
- net at L3.2, U11.8 (LX): now also D12.1
Changed lines of the file:
@@
 EESchema Schematic File Version 2
+LIBS:camprj_kicad-rescue
 LIBS:power
 LIBS:device
@@
 $Descr A4 11693 8268
 encoding utf-8
-Sheet 9 13
+Sheet 8 13
 Title ""
 Date ""
@@
 AR Path="/59604F02/59608776/59604F14" Ref="U14"  Part="1"
 AR Path="/59604F02/59608870/59604F14" Ref="U15"  Part="1"
-F 0 "U12" H 5750 2950 50  0000 C CNN
+F 0 "U15" H 5750 2950 50  0000 C CNN
 F 1 "MAX1561" H 5750 3150 50  0000 C CNN
 F 2 "SparkFun-PowerIC:8-TDFN-EP" H 5750 3050 50  0001 C CNN
@@
 AR Path="/59604F02/59608776/5960555F" Ref="C34"  Part="1"
 AR Path="/59604F02/59608870/5960555F" Ref="C37"  Part="1"
-F 0 "C28" H 4625 3750 50  0000 L CNN
+F 0 "C37" H 4625 3750 50  0000 L CNN
 F 1 "0.1uF" H 4625 3550 50  0000 L CNN
 F 2 "Capacitors_SMD:C_0603_HandSoldering" H 4638 3500 50  0001 C CNN
@@
 AR Path="/59604F02/59608776/5960566F" Ref="C33"  Part="1"
 AR Path="/59604F02/59608870/5960566F" Ref="C36"  Part="1"
-F 0 "C27" H 4425 2700 50  0000 L CNN
+F 0 "C36" H 4425 2700 50  0000 L CNN
 F 1 "2.2uF" H 4425 2500 50  0000 L CNN
 F 2 "Capacitors_SMD:C_0603_HandSoldering" H 4438 2450 50  0001 C CNN
@@
 AR Path="/59604F02/59608776/5960587B" Ref="C35"  Part="1"
 AR Path="/59604F02/59608870/5960587B" Ref="C38"  Part="1"
-F 0 "C29" H 7025 3050 50  0000 L CNN
+F 0 "C38" H 7025 3050 50  0000 L CNN
 F 1 "0.1uF" H 7025 2850 50  0000 L CNN
 F 2 "Capacitors_SMD:C_0603_HandSoldering" H 7038 2800 50  0001 C CNN
@@
 AR Path="/59604F02/59608776/59605DEA" Ref="L6"  Part="1"
 AR Path="/59604F02/59608870/59605DEA" Ref="L7"  Part="1"
-F 0 "L4" V 5550 2250 50  0000 C CNN
+F 0 "L7" V 5550 2250 50  0000 C CNN
 F 1 "47uH" V 5675 2250 50  0000 C CNN
 F 2 "Inductors_SMD:L_1210_HandSoldering" H 5600 2250 50  0001 C CNN
 F 3 "" H 5600 2250 50  0001 C CNN
 	1    5600 2250
-	0    -1   -1   0
-$EndComp
-$Comp
-L LEPTONCUSTOM_DIODE-SCHOTTKY-B340A D7
-U 1 1 59605EC3
-P 6750 2600
-AR Path="/59604F02/59607CD4/59605EC3" Ref="D7"  Part="1"
-AR Path="/59604F02/59604F09/59605EC3" Ref="D2"  Part="1"
-AR Path="/59604F02/5960845F/59605EC3" Ref="D12"  Part="1"
-AR Path="/59604F02/59608613/59605EC3" Ref="D17"  Part="1"
-AR Path="/59604F02/59608776/59605EC3" Ref="D22"  Part="1"
-AR Path="/59604F02/59608870/59605EC3" Ref="D27"  Part="1"
-F 0 "D12" H 6850 2619 45  0000 L BNN
-F 1 "B340A" H 6600 2650 45  0000 L BNN
-F 2 "Myfootprints:D_SMA_Handsoldering_AC" H 6780 2750 20  0001 C CNN
-F 3 "" H 6750 2600 60  0001 C CNN
-	1    6750 2600
 	0    -1   -1   0
 $EndComp
@@
 AR Path="/59604F02/59608776/59606309" Ref="D23"  Part="1"
 AR Path="/59604F02/59608870/59606309" Ref="D28"  Part="1"
-F 0 "D13" H 7600 2750 50  0000 C CNN
+F 0 "D28" H 7600 2750 50  0000 C CNN
 F 1 "LED" H 7600 2550 50  0000 C CNN
 F 2 "LEDs:LED_PLCC-2" H 7600 2650 50  0001 C CNN
@@
 AR Path="/59604F02/59608776/596063DB" Ref="D24"  Part="1"
 AR Path="/59604F02/59608870/596063DB" Ref="D29"  Part="1"
-F 0 "D14" H 7600 3150 50  0000 C CNN
+F 0 "D29" H 7600 3150 50  0000 C CNN
 F 1 "LED" H 7600 2950 50  0000 C CNN
 F 2 "LEDs:LED_PLCC-2" H 7600 3050 50  0001 C CNN
@@
 AR Path="/59604F02/59608776/596064A1" Ref="D25"  Part="1"
 AR Path="/59604F02/59608870/596064A1" Ref="D30"  Part="1"
-F 0 "D15" H 7600 3550 50  0000 C CNN
+F 0 "D30" H 7600 3550 50  0000 C CNN
 F 1 "LED" H 7600 3350 50  0000 C CNN
 F 2 "LEDs:LED_PLCC-2" H 7600 3450 50  0001 C CNN
@@
 AR Path="/59604F02/59608776/596064D7" Ref="D26"  Part="1"
 AR Path="/59604F02/59608870/596064D7" Ref="D31"  Part="1"
-F 0 "D16" H 7600 3950 50  0000 C CNN
+F 0 "D31" H 7600 3950 50  0000 C CNN
 F 1 "LED" H 7600 3750 50  0000 C CNN
 F 2 "LEDs:LED_PLCC-2" H 7600 3850 50  0001 C CNN
@@
 AR Path="/59604F02/59608776/59606544" Ref="R10"  Part="1"
 AR Path="/59604F02/59608870/59606544" Ref="R11"  Part="1"
-F 0 "R8" V 7680 4300 50  0000 C CNN
+F 0 "R11" V 7680 4300 50  0000 C CNN
 F 1 "7.5" V 7600 4300 50  0000 C CNN
 F 2 "Resistors_SMD:R_0603_HandSoldering" V 7530 4300 50  0001 C CNN
@@
 Text HLabel 4000 3100 0    60   Input ~ 0
 PWM_IN
+$Comp
+L CMDSH2-3 D12
+U 1 1 597479DB
+P 6750 2600
+AR Path="/59604F02/5960845F/597479DB" Ref="D12"  Part="1"
+AR Path="/59604F02/59604F09/597479DB" Ref="D2"  Part="1"
+AR Path="/59604F02/59607CD4/597479DB" Ref="D7"  Part="1"
+AR Path="/59604F02/59608613/597479DB" Ref="D17"  Part="1"
+AR Path="/59604F02/59608776/597479DB" Ref="D22"  Part="1"
+AR Path="/59604F02/59608870/597479DB" Ref="D27"  Part="1"
+F 0 "D27" H 6850 2619 45  0000 L BNN
+F 1 "CMDSH2-3" V 6750 2650 45  0000 L BNN
+F 2 "Diodes_SMD:D_SOD-323_HandSoldering" H 6780 2750 20  0001 C CNN
+F 3 "http://www.mouser.com/ds/2/68/cmdsh2-3-39086.pdf" H 6850 2619 60  0001 C CNN
+F 4 "http://www.mouser.ch/ProductDetail/Central-Semiconductor/CMDSH2-3-TR/?qs=AjE1biBnhWMUdOF9vZ5x%252bg==" H 6950 2719 60  0001 C CNN "Buy Link"
+	1    6750 2600
+	0    -1   -1   0
+$EndComp
 $EndSCHEMATC

Commit message: Final Delivery
Parts:
- D12: MPN (none) -> CMDSH2-3 TR
- U11: MPN (none) -> MAX1561ETA+T
Changed lines of the file:
@@
 $Descr A4 11693 8268
 encoding utf-8
-Sheet 8 13
-Title ""
-Date ""
-Rev ""
-Comp ""
-Comment1 ""
+Sheet 9 13
+Title "LED Driver"
+Date "2017-08-02"
+Rev "1"
+Comp "MHSL ETH Zurich"
+Comment1 "Geethan Karunaratne"
 Comment2 ""
 Comment3 ""
@@
 F 3 "http://www.mouser.com/ds/2/256/MAX1561-MAX1599-65829.pdf" H 5750 3050 50  0001 C CNN
 F 4 "http://www.mouser.ch/ProductDetail/Maxim-Integrated/MAX1561ETA+T/?qs=p6VZ%252bklCkRSw1RT%2f%2fPr34Q==" H 5750 3050 60  0001 C CNN "Buy Link"
+F 5 "MAX1561ETA+T" H 5750 3050 60  0001 C CNN "MPN"
 	1    5750 3050
 	1    0    0    -1
@@
 F 3 "http://www.mouser.com/ds/2/68/cmdsh2-3-39086.pdf" H 6850 2619 60  0001 C CNN
 F 4 "http://www.mouser.ch/ProductDetail/Central-Semiconductor/CMDSH2-3-TR/?qs=AjE1biBnhWMUdOF9vZ5x%252bg==" H 6950 2719 60  0001 C CNN "Buy Link"
+F 5 "CMDSH2-3 TR" H 6750 2600 60  0001 C CNN "MPN"
 	1    6750 2600
 	0    -1   -1   0
